Commit message: added move_base into the launch file

File: scooter_launch/urdf/scooter.urdf (robot description, URDF)
Before this commit: robot scooter, 7 links, 6 joints
Links:
- added link base_footprint
Joints:
- added joint footprint_joint: type fixed, parent base_link, child base_footprint, origin xyz=0 0 0 rpy=0 0 0
- joint laser_joint: origin xyz=0 0 0 rpy=0 0 0 -> xyz=0 0 0 rpy=0 0 -3.1415

Commit message: scooter_nav conflict resolved

File: scooter_launch/urdf/scooter.urdf (robot description, URDF)
Before this commit: robot scooter, 8 links, 7 joints
Links:
- removed link base_footprint
Joints:
- removed joint footprint_joint

Commit message: first demo

File: scooter_launch/urdf/scooter.urdf (robot description, URDF)
Before this commit: robot scooter, 7 links, 6 joints
Joints:
- joint laser_joint: origin xyz=0 0 0 rpy=0 0 -3.1415 -> xyz=1 0.1 0.1 rpy=0 0 -3.1415
- joint zed_camera_center_joint: origin xyz=0 0 0 rpy=0 0 0 -> xyz=0 0 1.6 rpy=0 0 0

Commit message: move

File: scooter_launch/urdf/scooter.urdf (robot description, URDF)
Before this commit: robot scooter, 7 links, 6 joints
Joints:
- joint zed_camera_center_joint: origin xyz=0 0 1.6 rpy=0 0 0 -> xyz=0 0 1.62 rpy=0 0 0
